File: keyboard.kicad_pcb (KiCad board)
At the start: 2 copper layers, 295 parts

Commit message: Update to plan
Parts:
- removed D_0, D_1, D_2, D_3, D_4, D_5, D_6, D_7, D_8, D_9, D_M1, D_M10, D_M2, D_M3, D_M4, D_M5, D_M6, D_M7, D_M8, D_M9, D_a1, D_app1, D_b1, D_brk1, D_bspc1, D_c1, D_comm1, D_d1, D_del1, D_dot1, D_down1, D_e1, D_end1, D_ent1, D_eql1, D_esc1, D_f1, D_f10, D_f11, D_f12, D_f13, D_f2, D_f3, D_f4, D_f5, D_f6, D_f7, D_f8, D_f9, D_g1, D_h1, D_home1, D_i1, D_ins1, D_j1, D_k1, D_l1, D_lalt1, D_lbrc1, D_lcps1, D_lctl1, D_left1, D_lgui1, D_lsft1, D_m11, D_mins1, D_n1, D_nubs1, D_o1, D_p1, D_pgdn1, D_pgup1, D_pscr1, D_q1, D_quot1, D_r1, D_ralt1, D_rbrc1, D_rctl1, D_re1, D_re2, D_rght1, D_rgui1, D_rsft1, D_s1, D_scln1, D_scrl1, D_slsh1, D_space1, D_t1, D_tab1, D_tilde1, D_u1, D_up1, D_v1, D_w1, D_x1, D_y1, D_z1: D_Small_Filled, Diode_SMD:D_0805_2012Metric_Pad1.15x1.40mm_HandSolder
- removed MX_M1, MX_M10, MX_M2, MX_M3, MX_M4, MX_M5, MX_M6, MX_M7, MX_M8, MX_M9, MX_brk1, MX_m11, MX_scrl1, MX_tilde1: MX-LED, 0_MX_Only:MXOnly-1U
- removed MX_lcps1: MX-LED, 0_MX_Only:MXOnly-1.75U
- removed MX_nubs1: MX-LED, 0_MX_Only:MXOnly-1.5U
- removed MX_space1: MX-LED, 0_MX_Only:MXOnly-6.25U-ReversedStabilizers
- removed R_0, R_1, R_2, R_3, R_4, R_5, R_6, R_7, R_8, R_9, R_M1, R_M10, R_M2, R_M3, R_M4, R_M5, R_M6, R_M7, R_M8, R_M9, R_a1, R_app1, R_b1, R_brk1, R_bspc1, R_c1, R_comm1, R_d1, R_del1, R_dot1, R_down1, R_e1, R_end1, R_ent1, R_eql1, R_esc1, R_f1, R_f10, R_f11, R_f12, R_f13, R_f2, R_f3, R_f4, R_f5, R_f6, R_f7, R_f8, R_f9, R_g1, R_h1, R_home1, R_i1, R_ins1, R_j1, R_k1, R_l1, R_lalt1, R_lbrc1, R_lcps1, R_lctl1, R_left1, R_lgui1, R_lsft1, R_m11, R_mins1, R_n1, R_nubs1, R_o1, R_p1, R_pgdn1, R_pgup1, R_pscr1, R_q1, R_quot1, R_r1, R_ralt1, R_rbrc1, R_rctl1, R_rght1, R_rgui1, R_rsft1, R_s1, R_scln1, R_scrl1, R_slsh1, R_space1, R_t1, R_tab1, R_tilde1, R_u1, R_up1, R_v1, R_w1, R_x1, R_y1, R_z1: R_Small, Resistor_SMD:R_0805_2012Metric_Pad1.20x1.40mm_HandSolder
- added MX_Macro1: MX-LED, 0_MX_Only:MXOnly-1U, F.Cu at (77.0, 155.6)
- added MX_Macro10: MX-LED, 0_MX_Only:MXOnly-1U, F.Cu at (96.0, 231.8)
- added MX_Macro2: MX-LED, 0_MX_Only:MXOnly-1U, F.Cu at (96.0, 155.6)
- added MX_Macro3: MX-LED, 0_MX_Only:MXOnly-1U, F.Cu at (77.0, 174.6)
- added MX_Macro4: MX-LED, 0_MX_Only:MXOnly-1U, F.Cu at (96.0, 174.6)
- added MX_Macro5: MX-LED, 0_MX_Only:MXOnly-1U, F.Cu at (77.0, 193.7)
- added MX_Macro6: MX-LED, 0_MX_Only:MXOnly-1U, F.Cu at (96.0, 193.7)
- added MX_Macro7: MX-LED, 0_MX_Only:MXOnly-1U, F.Cu at (77.0, 212.7)
- added MX_Macro8: MX-LED, 0_MX_Only:MXOnly-1U, F.Cu at (96.0, 212.7)
- added MX_Macro9: MX-LED, 0_MX_Only:MXOnly-1U, F.Cu at (77.0, 231.8)
- added MX_bsls1: MX-LED, 0_MX_Only:MXOnly-1.5U, F.Cu at (386.6, 174.6)
- added MX_caps1: MX-LED, 0_MX_Only:MXOnly-1.75U, F.Cu at (131.8, 193.7)
- added MX_grv1: MX-LED, 0_MX_Only:MXOnly-1U, F.Cu at (124.6, 155.6)
- added MX_m1: MX-LED, 0_MX_Only:MXOnly-1U, F.Cu at (281.8, 212.7)
- added MX_paus1: MX-LED, 0_MX_Only:MXOnly-1U, F.Cu at (458.0, 127.0)
- added MX_sclk1: MX-LED, 0_MX_Only:MXOnly-1U, F.Cu at (438.9, 127.0)
- added MX_spc1: MX-LED, 0_MX_Only:MXOnly-6.25U-ReversedStabilizers, F.Cu at (246.1, 231.8)
- added U1: Pico_TP, 0_MCU_RaspberryPi_and_Boards:RPi_Pico_SMD_TP, F.Cu at (41.1, 184.8)
- added USB1: HRO-TYPE-C-31-M-12, 0_Keebio:HRO-TYPE-C-31-M-12-Assembly, F.Cu at (51.6, 115.7)
- MX_bspc1: footprint 0_MX_Only:MXOnly-2U-ReversedStabilizers -> 0_MX_Only:MXOnly-2U
- MX_rgui1: footprint 0_MX_Only:MXOnly-1U -> 0_MX_Only:MXOnly-1.25U
- SW_re1, SW_re2: footprint keebio:RotaryEncoder_Alps_EC11E-Switch_Vertical_H20mm -> 0_Keebio:RotaryEncoder_EC11
- moved MX_pscr1 68.4 mm to (419.9, 127.0)
- moved SW_re2 51.2 mm to (77.0, 127.0)
- moved MX_f6 37.0 mm to (266.7, 126.2)
- moved MX_f7 37.0 mm to (285.8, 126.2)
- moved MX_f5 37.0 mm to (247.7, 126.2)
- moved MX_f8 37.0 mm to (304.8, 126.2)
- moved MX_f9 36.5 mm to (334.2, 126.2)
- moved MX_f4 36.5 mm to (219.1, 127.0)
- moved MX_f1 36.5 mm to (161.9, 127.0)
- moved MX_f2 36.5 mm to (181.0, 127.0)
- moved MX_f3 36.5 mm to (200.0, 127.0)
- moved MX_f10 36.5 mm to (353.2, 126.2)
- moved MX_f11 36.5 mm to (372.3, 126.2)
- moved MX_f12 36.5 mm to (391.3, 126.2)
- moved MX_esc1 35.9 mm to (124.6, 127.0)
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Connections:
- MX_0 pad 1: Col_13 -> unconnected-(MX_0-Pad1)
- MX_0 pad 3: Net-(MX_0-Pad3) -> LED_VIN
- MX_0 pad 4: LED_GND -> Net-(MX_0-Pad4)
- MX_1 pad 1: Col_4 -> unconnected-(MX_1-Pad1)
- MX_1 pad 3: Net-(MX_1-Pad3) -> LED_VIN
- MX_1 pad 4: LED_GND -> Net-(MX_1-Pad4)
- MX_2 pad 1: Col_5 -> unconnected-(MX_2-Pad1)
- MX_2 pad 3: Net-(MX_2-Pad3) -> LED_VIN
- MX_2 pad 4: LED_GND -> Net-(MX_2-Pad4)
- MX_3 pad 1: Col_6 -> unconnected-(MX_3-Pad1)
- MX_3 pad 3: Net-(MX_3-Pad3) -> LED_VIN
- MX_3 pad 4: LED_GND -> Net-(MX_3-Pad4)
- MX_4 pad 1: Col_7 -> unconnected-(MX_4-Pad1)
- MX_4 pad 3: Net-(MX_4-Pad3) -> LED_VIN
- MX_4 pad 4: LED_GND -> Net-(MX_4-Pad4)
- MX_5 pad 1: Col_8 -> unconnected-(MX_5-Pad1)
- MX_5 pad 3: Net-(MX_5-Pad3) -> LED_VIN
- MX_5 pad 4: LED_GND -> Net-(MX_5-Pad4)
- MX_6 pad 1: Col_9 -> unconnected-(MX_6-Pad1)
- MX_6 pad 3: Net-(MX_6-Pad3) -> LED_VIN
- MX_6 pad 4: LED_GND -> Net-(MX_6-Pad4)
- MX_7 pad 1: Col_10 -> unconnected-(MX_7-Pad1)
- MX_7 pad 3: Net-(MX_7-Pad3) -> LED_VIN
- MX_7 pad 4: LED_GND -> Net-(MX_7-Pad4)
- MX_8 pad 1: Col_11 -> unconnected-(MX_8-Pad1)
- MX_8 pad 3: Net-(MX_8-Pad3) -> LED_VIN
- MX_8 pad 4: LED_GND -> Net-(MX_8-Pad4)
- MX_9 pad 1: Col_12 -> unconnected-(MX_9-Pad1)
- MX_9 pad 3: Net-(MX_9-Pad3) -> LED_VIN
- MX_9 pad 4: LED_GND -> Net-(MX_9-Pad4)
- MX_a1 pad 1: Col_4 -> unconnected-(MX_a1-Pad1)
- MX_a1 pad 3: Net-(MX_a1-Pad3) -> LED_VIN
- MX_a1 pad 4: LED_GND -> Net-(MX_a1-Pad4)
- MX_app1 pad 1: Col_15 -> unconnected-(MX_app1-Pad1)
- MX_app1 pad 3: Net-(MX_app1-Pad3) -> LED_VIN
- MX_app1 pad 4: LED_GND -> Net-(MX_app1-Pad4)
- MX_b1 pad 1: Col_9 -> unconnected-(MX_b1-Pad1)
- MX_b1 pad 3: Net-(MX_b1-Pad3) -> LED_VIN
- MX_b1 pad 4: LED_GND -> Net-(MX_b1-Pad4)
- MX_bspc1 pad 1: Col_16 -> unconnected-(MX_bspc1-Pad1)
- MX_bspc1 pad 3: Net-(MX_bspc1-Pad3) -> LED_VIN
- MX_bspc1 pad 4: LED_GND -> Net-(MX_bspc1-Pad4)
- MX_c1 pad 1: Col_7 -> unconnected-(MX_c1-Pad1)
- MX_c1 pad 3: Net-(MX_c1-Pad3) -> LED_VIN
- MX_c1 pad 4: LED_GND -> Net-(MX_c1-Pad4)
- MX_comm1 pad 1: Col_12 -> unconnected-(MX_comm1-Pad1)
- MX_comm1 pad 3: Net-(MX_comm1-Pad3) -> LED_VIN
- MX_comm1 pad 4: LED_GND -> Net-(MX_comm1-Pad4)
- MX_d1 pad 1: Col_6 -> unconnected-(MX_d1-Pad1)
- MX_d1 pad 3: Net-(MX_d1-Pad3) -> LED_VIN
- MX_d1 pad 4: LED_GND -> Net-(MX_d1-Pad4)
- MX_del1 pad 1: Col_18 -> unconnected-(MX_del1-Pad1)
- MX_del1 pad 3: Net-(MX_del1-Pad3) -> LED_VIN
- MX_del1 pad 4: LED_GND -> Net-(MX_del1-Pad4)
- MX_dot1 pad 1: Col_13 -> unconnected-(MX_dot1-Pad1)
- MX_dot1 pad 3: Net-(MX_dot1-Pad3) -> LED_VIN
- MX_dot1 pad 4: LED_GND -> Net-(MX_dot1-Pad4)
- MX_down1 pad 1: Col_19 -> unconnected-(MX_down1-Pad1)
- MX_down1 pad 3: Net-(MX_down1-Pad3) -> LED_VIN
- MX_down1 pad 4: LED_GND -> Net-(MX_down1-Pad4)
- MX_e1 pad 1: Col_6 -> unconnected-(MX_e1-Pad1)
- MX_e1 pad 3: Net-(MX_e1-Pad3) -> LED_VIN
- MX_e1 pad 4: LED_GND -> Net-(MX_e1-Pad4)
- MX_end1 pad 1: Col_19 -> unconnected-(MX_end1-Pad1)
- MX_end1 pad 3: Net-(MX_end1-Pad3) -> LED_VIN
- MX_end1 pad 4: LED_GND -> Net-(MX_end1-Pad4)
- MX_ent1 pad 1: Col_16 -> unconnected-(MX_ent1-Pad1)
- MX_ent1 pad 3: Net-(MX_ent1-Pad3) -> LED_VIN
- MX_ent1 pad 4: LED_GND -> Net-(MX_ent1-Pad4)
- MX_eql1 pad 1: Col_15 -> unconnected-(MX_eql1-Pad1)
- MX_eql1 pad 3: Net-(MX_eql1-Pad3) -> LED_VIN
- MX_eql1 pad 4: LED_GND -> Net-(MX_eql1-Pad4)
- MX_esc1 pad 1: Col_3 -> unconnected-(MX_esc1-Pad1)
- MX_esc1 pad 3: Net-(MX_esc1-Pad3) -> LED_VIN
- MX_esc1 pad 4: LED_GND -> Net-(MX_esc1-Pad4)
- MX_f1 pad 1: Col_5 -> unconnected-(MX_f1-Pad1)
- MX_f1 pad 3: Net-(MX_f1-Pad3) -> LED_VIN
- MX_f1 pad 4: LED_GND -> Net-(MX_f1-Pad4)
- MX_f10 pad 1: Col_14 -> unconnected-(MX_f10-Pad1)
- MX_f10 pad 3: Net-(MX_f10-Pad3) -> LED_VIN
- MX_f10 pad 4: LED_GND -> Net-(MX_f10-Pad4)
- MX_f11 pad 1: Col_15 -> unconnected-(MX_f11-Pad1)
- MX_f11 pad 3: Net-(MX_f11-Pad3) -> LED_VIN
- MX_f11 pad 4: LED_GND -> Net-(MX_f11-Pad4)
- MX_f12 pad 1: Col_16 -> unconnected-(MX_f12-Pad1)
- MX_f12 pad 3: Net-(MX_f12-Pad3) -> LED_VIN
- MX_f12 pad 4: LED_GND -> Net-(MX_f12-Pad4)
- MX_f13 pad 1: Col_7 -> unconnected-(MX_f13-Pad1)
- MX_f13 pad 3: Net-(MX_f13-Pad3) -> LED_VIN
- MX_f13 pad 4: LED_GND -> Net-(MX_f13-Pad4)
- MX_f2 pad 1: Col_6 -> unconnected-(MX_f2-Pad1)
- MX_f2 pad 3: Net-(MX_f2-Pad3) -> LED_VIN
- MX_f2 pad 4: LED_GND -> Net-(MX_f2-Pad4)
- MX_f3 pad 1: Col_7 -> unconnected-(MX_f3-Pad1)
- MX_f3 pad 3: Net-(MX_f3-Pad3) -> LED_VIN
- MX_f3 pad 4: LED_GND -> Net-(MX_f3-Pad4)
- MX_f4 pad 1: Col_8 -> unconnected-(MX_f4-Pad1)
- MX_f4 pad 3: Net-(MX_f4-Pad3) -> LED_VIN
- MX_f4 pad 4: LED_GND -> Net-(MX_f4-Pad4)
- MX_f5 pad 1: Col_9 -> unconnected-(MX_f5-Pad1)
- MX_f5 pad 3: Net-(MX_f5-Pad3) -> LED_VIN
- MX_f5 pad 4: LED_GND -> Net-(MX_f5-Pad4)
- MX_f6 pad 1: Col_10 -> unconnected-(MX_f6-Pad1)
- MX_f6 pad 3: Net-(MX_f6-Pad3) -> LED_VIN
- MX_f6 pad 4: LED_GND -> Net-(MX_f6-Pad4)
- MX_f7 pad 1: Col_11 -> unconnected-(MX_f7-Pad1)
- MX_f7 pad 3: Net-(MX_f7-Pad3) -> LED_VIN
- MX_f7 pad 4: LED_GND -> Net-(MX_f7-Pad4)
- MX_f8 pad 1: Col_12 -> unconnected-(MX_f8-Pad1)
- MX_f8 pad 3: Net-(MX_f8-Pad3) -> LED_VIN
- MX_f8 pad 4: LED_GND -> Net-(MX_f8-Pad4)
- MX_f9 pad 1: Col_13 -> unconnected-(MX_f9-Pad1)
- MX_f9 pad 3: Net-(MX_f9-Pad3) -> LED_VIN
- MX_f9 pad 4: LED_GND -> Net-(MX_f9-Pad4)
- MX_g1 pad 1: Col_8 -> unconnected-(MX_g1-Pad1)
- MX_g1 pad 3: Net-(MX_g1-Pad3) -> LED_VIN
- MX_g1 pad 4: LED_GND -> Net-(MX_g1-Pad4)
- MX_h1 pad 1: Col_9 -> unconnected-(MX_h1-Pad1)
- MX_h1 pad 3: Net-(MX_h1-Pad3) -> LED_VIN
- MX_h1 pad 4: LED_GND -> Net-(MX_h1-Pad4)
- MX_home1 pad 1: Col_19 -> unconnected-(MX_home1-Pad1)
- MX_home1 pad 3: Net-(MX_home1-Pad3) -> LED_VIN
- MX_home1 pad 4: LED_GND -> Net-(MX_home1-Pad4)
- MX_i1 pad 1: Col_11 -> unconnected-(MX_i1-Pad1)
- MX_i1 pad 3: Net-(MX_i1-Pad3) -> LED_VIN
- MX_i1 pad 4: LED_GND -> Net-(MX_i1-Pad4)
- MX_ins1 pad 1: Col_18 -> unconnected-(MX_ins1-Pad1)
- MX_ins1 pad 3: Net-(MX_ins1-Pad3) -> LED_VIN
- MX_ins1 pad 4: LED_GND -> Net-(MX_ins1-Pad4)
- MX_j1 pad 1: Col_10 -> unconnected-(MX_j1-Pad1)
- MX_j1 pad 3: Net-(MX_j1-Pad3) -> LED_VIN
- MX_j1 pad 4: LED_GND -> Net-(MX_j1-Pad4)
- MX_k1 pad 1: Col_11 -> unconnected-(MX_k1-Pad1)
- MX_k1 pad 3: Net-(MX_k1-Pad3) -> LED_VIN
- MX_k1 pad 4: LED_GND -> Net-(MX_k1-Pad4)
- MX_l1 pad 1: Col_12 -> unconnected-(MX_l1-Pad1)
- MX_l1 pad 3: Net-(MX_l1-Pad3) -> LED_VIN
- MX_l1 pad 4: LED_GND -> Net-(MX_l1-Pad4)
- MX_lalt1 pad 1: Col_5 -> unconnected-(MX_lalt1-Pad1)
- MX_lalt1 pad 3: Net-(MX_lalt1-Pad3) -> LED_VIN
- MX_lalt1 pad 4: LED_GND -> Net-(MX_lalt1-Pad4)
- MX_lbrc1 pad 1: Col_14 -> unconnected-(MX_lbrc1-Pad1)
- MX_lbrc1 pad 3: Net-(MX_lbrc1-Pad3) -> LED_VIN
- MX_lbrc1 pad 4: LED_GND -> Net-(MX_lbrc1-Pad4)
- MX_lctl1 pad 1: Col_3 -> unconnected-(MX_lctl1-Pad1)
- MX_lctl1 pad 3: Net-(MX_lctl1-Pad3) -> LED_VIN
- MX_lctl1 pad 4: LED_GND -> Net-(MX_lctl1-Pad4)
- MX_left1 pad 1: Col_18 -> unconnected-(MX_left1-Pad1)
- MX_left1 pad 3: Net-(MX_left1-Pad3) -> LED_VIN
- MX_left1 pad 4: LED_GND -> Net-(MX_left1-Pad4)
- MX_lgui1 pad 1: Col_4 -> unconnected-(MX_lgui1-Pad1)
- MX_lgui1 pad 3: Net-(MX_lgui1-Pad3) -> LED_VIN
- MX_lgui1 pad 4: LED_GND -> Net-(MX_lgui1-Pad4)
- MX_lsft1 pad 1: Col_3 -> unconnected-(MX_lsft1-Pad1)
- MX_lsft1 pad 3: Net-(MX_lsft1-Pad3) -> LED_VIN
- MX_lsft1 pad 4: LED_GND -> Net-(MX_lsft1-Pad4)
- MX_mins1 pad 1: Col_14 -> unconnected-(MX_mins1-Pad1)
- MX_mins1 pad 3: Net-(MX_mins1-Pad3) -> LED_VIN
- MX_mins1 pad 4: LED_GND -> Net-(MX_mins1-Pad4)
- MX_n1 pad 1: Col_10 -> unconnected-(MX_n1-Pad1)
- MX_n1 pad 3: Net-(MX_n1-Pad3) -> LED_VIN
- MX_n1 pad 4: LED_GND -> Net-(MX_n1-Pad4)
- MX_o1 pad 1: Col_12 -> unconnected-(MX_o1-Pad1)
- MX_o1 pad 3: Net-(MX_o1-Pad3) -> LED_VIN
- MX_o1 pad 4: LED_GND -> Net-(MX_o1-Pad4)
- MX_p1 pad 1: Col_13 -> unconnected-(MX_p1-Pad1)
- MX_p1 pad 3: Net-(MX_p1-Pad3) -> LED_VIN
- MX_p1 pad 4: LED_GND -> Net-(MX_p1-Pad4)
- MX_pgdn1 pad 1: Col_20 -> unconnected-(MX_pgdn1-Pad1)
- MX_pgdn1 pad 3: Net-(MX_pgdn1-Pad3) -> LED_VIN
- MX_pgdn1 pad 4: LED_GND -> Net-(MX_pgdn1-Pad4)
- MX_pgup1 pad 1: Col_20 -> unconnected-(MX_pgup1-Pad1)
- MX_pgup1 pad 3: Net-(MX_pgup1-Pad3) -> LED_VIN
- MX_pgup1 pad 4: LED_GND -> Net-(MX_pgup1-Pad4)
- MX_pscr1 pad 1: Col_18 -> unconnected-(MX_pscr1-Pad1)
- MX_pscr1 pad 3: Net-(MX_pscr1-Pad3) -> LED_VIN
- MX_pscr1 pad 4: LED_GND -> Net-(MX_pscr1-Pad4)
- MX_q1 pad 1: Col_4 -> unconnected-(MX_q1-Pad1)
- MX_q1 pad 3: Net-(MX_q1-Pad3) -> LED_VIN
- MX_q1 pad 4: LED_GND -> Net-(MX_q1-Pad4)
- MX_quot1 pad 1: Col_14 -> unconnected-(MX_quot1-Pad1)
- MX_quot1 pad 3: Net-(MX_quot1-Pad3) -> LED_VIN
- MX_quot1 pad 4: LED_GND -> Net-(MX_quot1-Pad4)
- MX_r1 pad 1: Col_7 -> unconnected-(MX_r1-Pad1)
- MX_r1 pad 3: Net-(MX_r1-Pad3) -> LED_VIN
- MX_r1 pad 4: LED_GND -> Net-(MX_r1-Pad4)
- MX_ralt1 pad 1: Col_13 -> unconnected-(MX_ralt1-Pad1)
- MX_ralt1 pad 3: Net-(MX_ralt1-Pad3) -> LED_VIN
- MX_ralt1 pad 4: LED_GND -> Net-(MX_ralt1-Pad4)
- MX_rbrc1 pad 1: Col_15 -> unconnected-(MX_rbrc1-Pad1)
- MX_rbrc1 pad 3: Net-(MX_rbrc1-Pad3) -> LED_VIN
- MX_rbrc1 pad 4: LED_GND -> Net-(MX_rbrc1-Pad4)
- MX_rctl1 pad 1: Col_16 -> unconnected-(MX_rctl1-Pad1)
- MX_rctl1 pad 3: Net-(MX_rctl1-Pad3) -> LED_VIN
- MX_rctl1 pad 4: LED_GND -> Net-(MX_rctl1-Pad4)
- MX_rght1 pad 1: Col_20 -> unconnected-(MX_rght1-Pad1)
- MX_rght1 pad 3: Net-(MX_rght1-Pad3) -> LED_VIN
- MX_rght1 pad 4: LED_GND -> Net-(MX_rght1-Pad4)
- MX_rgui1 pad 1: Col_14 -> unconnected-(MX_rgui1-Pad1)
- MX_rgui1 pad 3: Net-(MX_rgui1-Pad3) -> LED_VIN
- MX_rgui1 pad 4: LED_GND -> Net-(MX_rgui1-Pad4)
- MX_rsft1 pad 1: Col_16 -> unconnected-(MX_rsft1-Pad1)
- MX_rsft1 pad 3: Net-(MX_rsft1-Pad3) -> LED_VIN
- MX_rsft1 pad 4: LED_GND -> Net-(MX_rsft1-Pad4)
- MX_s1 pad 1: Col_5 -> unconnected-(MX_s1-Pad1)
- MX_s1 pad 3: Net-(MX_s1-Pad3) -> LED_VIN
- MX_s1 pad 4: LED_GND -> Net-(MX_s1-Pad4)
- MX_scln1 pad 1: Col_13 -> unconnected-(MX_scln1-Pad1)
- MX_scln1 pad 3: Net-(MX_scln1-Pad3) -> LED_VIN
- MX_scln1 pad 4: LED_GND -> Net-(MX_scln1-Pad4)
- MX_slsh1 pad 1: Col_14 -> unconnected-(MX_slsh1-Pad1)
- MX_slsh1 pad 3: Net-(MX_slsh1-Pad3) -> LED_VIN
- MX_slsh1 pad 4: LED_GND -> Net-(MX_slsh1-Pad4)
- MX_t1 pad 1: Col_8 -> unconnected-(MX_t1-Pad1)
- MX_t1 pad 3: Net-(MX_t1-Pad3) -> LED_VIN
- MX_t1 pad 4: LED_GND -> Net-(MX_t1-Pad4)
- MX_tab1 pad 1: Col_3 -> unconnected-(MX_tab1-Pad1)
- MX_tab1 pad 3: Net-(MX_tab1-Pad3) -> LED_VIN
- MX_tab1 pad 4: LED_GND -> Net-(MX_tab1-Pad4)
- MX_u1 pad 1: Col_10 -> unconnected-(MX_u1-Pad1)
- MX_u1 pad 3: Net-(MX_u1-Pad3) -> LED_VIN
- MX_u1 pad 4: LED_GND -> Net-(MX_u1-Pad4)
- MX_up1 pad 1: Col_19 -> unconnected-(MX_up1-Pad1)
- MX_up1 pad 3: Net-(MX_up1-Pad3) -> LED_VIN
- MX_up1 pad 4: LED_GND -> Net-(MX_up1-Pad4)
- MX_v1 pad 1: Col_8 -> unconnected-(MX_v1-Pad1)
- MX_v1 pad 3: Net-(MX_v1-Pad3) -> LED_VIN
- MX_v1 pad 4: LED_GND -> Net-(MX_v1-Pad4)
- MX_w1 pad 1: Col_5 -> unconnected-(MX_w1-Pad1)
- MX_w1 pad 3: Net-(MX_w1-Pad3) -> LED_VIN
- MX_w1 pad 4: LED_GND -> Net-(MX_w1-Pad4)
- MX_x1 pad 1: Col_6 -> unconnected-(MX_x1-Pad1)
- MX_x1 pad 3: Net-(MX_x1-Pad3) -> LED_VIN
- MX_x1 pad 4: LED_GND -> Net-(MX_x1-Pad4)
- MX_y1 pad 1: Col_9 -> unconnected-(MX_y1-Pad1)
- MX_y1 pad 3: Net-(MX_y1-Pad3) -> LED_VIN
- MX_y1 pad 4: LED_GND -> Net-(MX_y1-Pad4)
- MX_z1 pad 1: Col_5 -> unconnected-(MX_z1-Pad1)
- MX_z1 pad 3: Net-(MX_z1-Pad3) -> LED_VIN
- MX_z1 pad 4: LED_GND -> Net-(MX_z1-Pad4)
- SW_re1 pad S2: Net-(D_re1-Pad2) -> Row_0
- SW_re2 pad S2: Net-(D_re2-Pad2) -> Row_0

Commit message: Keyboard
Parts:
- added D_0: D_Small, Diode_SMD:D_0805_2012Metric_Pad1.15x1.40mm_HandSolder, B.Cu at (323.1, 148.4)
- added D_1: D_Small, Diode_SMD:D_0805_2012Metric_Pad1.15x1.40mm_HandSolder, B.Cu at (151.6, 148.4)
- added D_2: D_Small, Diode_SMD:D_0805_2012Metric_Pad1.15x1.40mm_HandSolder, B.Cu at (170.7, 148.4)
- added D_3: D_Small, Diode_SMD:D_0805_2012Metric_Pad1.15x1.40mm_HandSolder, B.Cu at (189.7, 148.4)
- added D_4: D_Small, Diode_SMD:D_0805_2012Metric_Pad1.15x1.40mm_HandSolder, B.Cu at (208.8, 148.4)
- added D_5: D_Small, Diode_SMD:D_0805_2012Metric_Pad1.15x1.40mm_HandSolder, B.Cu at (227.8, 148.4)
- added D_6: D_Small, Diode_SMD:D_0805_2012Metric_Pad1.15x1.40mm_HandSolder, B.Cu at (246.9, 148.4)
- added D_7: D_Small, Diode_SMD:D_0805_2012Metric_Pad1.15x1.40mm_HandSolder, B.Cu at (265.9, 148.4)
- added D_8: D_Small, Diode_SMD:D_0805_2012Metric_Pad1.15x1.40mm_HandSolder, B.Cu at (285.0, 148.4)
- added D_9: D_Small, Diode_SMD:D_0805_2012Metric_Pad1.15x1.40mm_HandSolder, B.Cu at (304.0, 148.4)
- added D_Macro1: D_Small, Diode_SMD:D_0805_2012Metric_Pad1.15x1.40mm_HandSolder, B.Cu at (84.9, 148.4)
- added D_Macro10: D_Small, Diode_SMD:D_0805_2012Metric_Pad1.15x1.40mm_HandSolder, B.Cu at (104.0, 224.6)
- added D_Macro2: D_Small, Diode_SMD:D_0805_2012Metric_Pad1.15x1.40mm_HandSolder, B.Cu at (104.0, 148.4)
- added D_Macro3: D_Small, Diode_SMD:D_0805_2012Metric_Pad1.15x1.40mm_HandSolder, B.Cu at (84.9, 167.5)
- added D_Macro4: D_Small, Diode_SMD:D_0805_2012Metric_Pad1.15x1.40mm_HandSolder, B.Cu at (104.0, 167.5)
- added D_Macro5: D_Small, Diode_SMD:D_0805_2012Metric_Pad1.15x1.40mm_HandSolder, B.Cu at (84.9, 186.5)
- added D_Macro6: D_Small, Diode_SMD:D_0805_2012Metric_Pad1.15x1.40mm_HandSolder, B.Cu at (104.0, 186.5)
- added D_Macro7: D_Small, Diode_SMD:D_0805_2012Metric_Pad1.15x1.40mm_HandSolder, B.Cu at (84.9, 205.6)
- added D_Macro8: D_Small, Diode_SMD:D_0805_2012Metric_Pad1.15x1.40mm_HandSolder, B.Cu at (104.0, 205.6)
- added D_Macro9: D_Small, Diode_SMD:D_0805_2012Metric_Pad1.15x1.40mm_HandSolder, B.Cu at (84.9, 224.6)
- added D_a1: D_Small, Diode_SMD:D_0805_2012Metric_Pad1.15x1.40mm_HandSolder, B.Cu at (165.9, 186.5)
- added D_app1: D_Small, Diode_SMD:D_0805_2012Metric_Pad1.15x1.40mm_HandSolder, B.Cu at (373.1, 224.6)
- added D_b1: D_Small, Diode_SMD:D_0805_2012Metric_Pad1.15x1.40mm_HandSolder, B.Cu at (251.6, 205.6)
- added D_bsls1: D_Small, Diode_SMD:D_0805_2012Metric_Pad1.15x1.40mm_HandSolder, B.Cu at (381.0, 167.5)
- added D_bspc1: D_Small, Diode_SMD:D_0805_2012Metric_Pad1.15x1.40mm_HandSolder, B.Cu at (389.7, 148.4)
- added D_c1: D_Small, Diode_SMD:D_0805_2012Metric_Pad1.15x1.40mm_HandSolder, B.Cu at (213.5, 205.6)
- added D_caps1: D_Small, Diode_SMD:D_0805_2012Metric_Pad1.15x1.40mm_HandSolder, B.Cu at (139.7, 186.5)
- added D_comm1: D_Small, Diode_SMD:D_0805_2012Metric_Pad1.15x1.40mm_HandSolder, B.Cu at (308.8, 205.6)
- added D_d1: D_Small, Diode_SMD:D_0805_2012Metric_Pad1.15x1.40mm_HandSolder, B.Cu at (204.0, 186.5)
- added D_del1: D_Small, Diode_SMD:D_0805_2012Metric_Pad1.15x1.40mm_HandSolder, B.Cu at (427.8, 167.5)
- added D_dot1: D_Small, Diode_SMD:D_0805_2012Metric_Pad1.15x1.40mm_HandSolder, B.Cu at (327.8, 205.6)
- added D_down1: D_Small, Diode_SMD:D_0805_2012Metric_Pad1.15x1.40mm_HandSolder, B.Cu at (446.9, 224.6)
- added D_e1: D_Small, Diode_SMD:D_0805_2012Metric_Pad1.15x1.40mm_HandSolder, B.Cu at (199.2, 167.5)
- added D_end1: D_Small, Diode_SMD:D_0805_2012Metric_Pad1.15x1.40mm_HandSolder, B.Cu at (446.9, 167.5)
- added D_ent1: D_Small, Diode_SMD:D_0805_2012Metric_Pad1.15x1.40mm_HandSolder, B.Cu at (387.4, 186.5)
- added D_eql1: D_Small, Diode_SMD:D_0805_2012Metric_Pad1.15x1.40mm_HandSolder, B.Cu at (361.2, 148.4)
- added D_esc1: D_Small, Diode_SMD:D_0805_2012Metric_Pad1.15x1.40mm_HandSolder, B.Cu at (132.6, 119.9)
- added D_f1: D_Small, Diode_SMD:D_0805_2012Metric_Pad1.15x1.40mm_HandSolder, B.Cu at (170.7, 119.9)
- added D_f10: D_Small, Diode_SMD:D_0805_2012Metric_Pad1.15x1.40mm_HandSolder, B.Cu at (361.2, 119.9)
- added D_f11: D_Small, Diode_SMD:D_0805_2012Metric_Pad1.15x1.40mm_HandSolder, B.Cu at (380.2, 119.9)
- added D_f12: D_Small, Diode_SMD:D_0805_2012Metric_Pad1.15x1.40mm_HandSolder, B.Cu at (399.3, 119.9)
- added D_f13: D_Small, Diode_SMD:D_0805_2012Metric_Pad1.15x1.40mm_HandSolder, B.Cu at (223.0, 186.5)
- added D_f2: D_Small, Diode_SMD:D_0805_2012Metric_Pad1.15x1.40mm_HandSolder, B.Cu at (189.7, 119.9)
- added D_f3: D_Small, Diode_SMD:D_0805_2012Metric_Pad1.15x1.40mm_HandSolder, B.Cu at (208.8, 119.9)
- added D_f4: D_Small, Diode_SMD:D_0805_2012Metric_Pad1.15x1.40mm_HandSolder, B.Cu at (227.8, 119.9)
- added D_f5: D_Small, Diode_SMD:D_0805_2012Metric_Pad1.15x1.40mm_HandSolder, B.Cu at (256.4, 119.9)
- added D_f6: D_Small, Diode_SMD:D_0805_2012Metric_Pad1.15x1.40mm_HandSolder, B.Cu at (275.4, 119.9)
- added D_f7: D_Small, Diode_SMD:D_0805_2012Metric_Pad1.15x1.40mm_HandSolder, B.Cu at (295.3, 119.9)
- added D_f8: D_Small, Diode_SMD:D_0805_2012Metric_Pad1.15x1.40mm_HandSolder, B.Cu at (313.5, 119.9)
- added D_f9: D_Small, Diode_SMD:D_0805_2012Metric_Pad1.15x1.40mm_HandSolder, B.Cu at (342.1, 119.9)
- added D_g1: D_Small, Diode_SMD:D_0805_2012Metric_Pad1.15x1.40mm_HandSolder, B.Cu at (242.1, 186.5)
- added D_grv1: D_Small, Diode_SMD:D_0805_2012Metric_Pad1.15x1.40mm_HandSolder, B.Cu at (132.6, 148.4)
- added D_h1: D_Small, Diode_SMD:D_0805_2012Metric_Pad1.15x1.40mm_HandSolder, B.Cu at (261.1, 186.5)
- added D_home1: D_Small, Diode_SMD:D_0805_2012Metric_Pad1.15x1.40mm_HandSolder, B.Cu at (446.9, 148.4)
- added D_i1: D_Small, Diode_SMD:D_0805_2012Metric_Pad1.15x1.40mm_HandSolder, B.Cu at (294.5, 167.5)
- added D_ins1: D_Small, Diode_SMD:D_0805_2012Metric_Pad1.15x1.40mm_HandSolder, B.Cu at (427.8, 148.4)
- added D_j1: D_Small, Diode_SMD:D_0805_2012Metric_Pad1.15x1.40mm_HandSolder, B.Cu at (280.2, 186.5)
- added D_k1: D_Small, Diode_SMD:D_0805_2012Metric_Pad1.15x1.40mm_HandSolder, B.Cu at (299.2, 186.5)
- added D_l1: D_Small, Diode_SMD:D_0805_2012Metric_Pad1.15x1.40mm_HandSolder, B.Cu at (318.3, 186.5)
- added D_lalt1: D_Small, Diode_SMD:D_0805_2012Metric_Pad1.15x1.40mm_HandSolder, B.Cu at (182.6, 224.6)
- added D_lbrc1: D_Small, Diode_SMD:D_0805_2012Metric_Pad1.15x1.40mm_HandSolder, B.Cu at (351.6, 167.5)
- added D_lctl1: D_Small, Diode_SMD:D_0805_2012Metric_Pad1.15x1.40mm_HandSolder, B.Cu at (134.9, 224.6)
- added D_left1: D_Small, Diode_SMD:D_0805_2012Metric_Pad1.15x1.40mm_HandSolder, B.Cu at (427.8, 224.6)
- added D_lgui1: D_Small, Diode_SMD:D_0805_2012Metric_Pad1.15x1.40mm_HandSolder, B.Cu at (158.8, 224.6)
- added D_lsft1: D_Small, Diode_SMD:D_0805_2012Metric_Pad1.15x1.40mm_HandSolder, B.Cu at (144.5, 205.6)
- added D_m1: D_Small, Diode_SMD:D_0805_2012Metric_Pad1.15x1.40mm_HandSolder, B.Cu at (289.7, 205.6)
- added D_mins1: D_Small, Diode_SMD:D_0805_2012Metric_Pad1.15x1.40mm_HandSolder, B.Cu at (342.1, 148.4)
- added D_n1: D_Small, Diode_SMD:D_0805_2012Metric_Pad1.15x1.40mm_HandSolder, B.Cu at (270.7, 205.6)
- added D_o1: D_Small, Diode_SMD:D_0805_2012Metric_Pad1.15x1.40mm_HandSolder, B.Cu at (313.5, 167.5)
- added D_p1: D_Small, Diode_SMD:D_0805_2012Metric_Pad1.15x1.40mm_HandSolder, B.Cu at (332.6, 167.5)
- added D_paus1: D_Small, Diode_SMD:D_0805_2012Metric_Pad1.15x1.40mm_HandSolder, B.Cu at (465.9, 119.9)
- added D_pgdn1: D_Small, Diode_SMD:D_0805_2012Metric_Pad1.15x1.40mm_HandSolder, B.Cu at (465.9, 167.5)
- added D_pgup1: D_Small, Diode_SMD:D_0805_2012Metric_Pad1.15x1.40mm_HandSolder, B.Cu at (465.9, 148.4)
- added D_pscr1: D_Small, Diode_SMD:D_0805_2012Metric_Pad1.15x1.40mm_HandSolder, B.Cu at (427.8, 119.9)
- added D_q1: D_Small, Diode_SMD:D_0805_2012Metric_Pad1.15x1.40mm_HandSolder, B.Cu at (161.1, 167.5)
- added D_quot1: D_Small, Diode_SMD:D_0805_2012Metric_Pad1.15x1.40mm_HandSolder, B.Cu at (356.4, 186.5)
- added D_r1: D_Small, Diode_SMD:D_0805_2012Metric_Pad1.15x1.40mm_HandSolder, B.Cu at (218.3, 167.5)
- added D_ralt1: D_Small, Diode_SMD:D_0805_2012Metric_Pad1.15x1.40mm_HandSolder, B.Cu at (325.4, 224.6)
- added D_rbrc1: D_Small, Diode_SMD:D_0805_2012Metric_Pad1.15x1.40mm_HandSolder, B.Cu at (373.9, 167.5)
- added D_rctl1: D_Small, Diode_SMD:D_0805_2012Metric_Pad1.15x1.40mm_HandSolder, B.Cu at (396.9, 224.6)
- added D_re1: D_Small, Diode_SMD:D_0805_2012Metric_Pad1.15x1.40mm_HandSolder, B.Cu at (70.6, 119.9)
- added D_re2: D_Small, Diode_SMD:D_0805_2012Metric_Pad1.15x1.40mm_HandSolder, B.Cu at (89.5, 119.9)
- added D_rght1: D_Small, Diode_SMD:D_0805_2012Metric_Pad1.15x1.40mm_HandSolder, B.Cu at (465.9, 224.6)
- added D_rgui1: D_Small, Diode_SMD:D_0805_2012Metric_Pad1.15x1.40mm_HandSolder, B.Cu at (349.2, 224.6)
- added D_rsft1: D_Small, Diode_SMD:D_0805_2012Metric_Pad1.15x1.40mm_HandSolder, B.Cu at (382.6, 205.6)
- added D_s1: D_Small, Diode_SMD:D_0805_2012Metric_Pad1.15x1.40mm_HandSolder, B.Cu at (184.9, 186.5)
- added D_sclk1: D_Small, Diode_SMD:D_0805_2012Metric_Pad1.15x1.40mm_HandSolder, B.Cu at (446.9, 119.9)
- added D_scln1: D_Small, Diode_SMD:D_0805_2012Metric_Pad1.15x1.40mm_HandSolder, B.Cu at (337.3, 186.5)
- added D_slsh1: D_Small, Diode_SMD:D_0805_2012Metric_Pad1.15x1.40mm_HandSolder, B.Cu at (346.9, 205.6)
- added D_spc1: D_Small, Diode_SMD:D_0805_2012Metric_Pad1.15x1.40mm_HandSolder, B.Cu at (254.0, 224.6)
- added D_t1: D_Small, Diode_SMD:D_0805_2012Metric_Pad1.15x1.40mm_HandSolder, B.Cu at (237.3, 167.5)
- added D_tab1: D_Small, Diode_SMD:D_0805_2012Metric_Pad1.15x1.40mm_HandSolder, B.Cu at (137.3, 167.5)
- added D_u1: D_Small, Diode_SMD:D_0805_2012Metric_Pad1.15x1.40mm_HandSolder, B.Cu at (275.4, 167.5)
- added D_up1: D_Small, Diode_SMD:D_0805_2012Metric_Pad1.15x1.40mm_HandSolder, B.Cu at (446.9, 205.6)
- added D_v1: D_Small, Diode_SMD:D_0805_2012Metric_Pad1.15x1.40mm_HandSolder, B.Cu at (232.6, 205.6)
- added D_w1: D_Small, Diode_SMD:D_0805_2012Metric_Pad1.15x1.40mm_HandSolder, B.Cu at (180.2, 167.5)
- added D_x1: D_Small, Diode_SMD:D_0805_2012Metric_Pad1.15x1.40mm_HandSolder, B.Cu at (194.5, 205.6)
- added D_y1: D_Small, Diode_SMD:D_0805_2012Metric_Pad1.15x1.40mm_HandSolder, B.Cu at (256.4, 167.5)
- added D_z1: D_Small, Diode_SMD:D_0805_2012Metric_Pad1.15x1.40mm_HandSolder, B.Cu at (175.4, 205.6)
- added R_0: R, Resistor_SMD:R_0805_2012Metric_Pad1.20x1.40mm_HandSolder, B.Cu at (323.1, 162.7)
- added R_1: R, Resistor_SMD:R_0805_2012Metric_Pad1.20x1.40mm_HandSolder, B.Cu at (151.6, 162.7)
- added R_2: R, Resistor_SMD:R_0805_2012Metric_Pad1.20x1.40mm_HandSolder, B.Cu at (170.7, 162.7)
- added R_3: R, Resistor_SMD:R_0805_2012Metric_Pad1.20x1.40mm_HandSolder, B.Cu at (189.7, 162.7)
- added R_4: R, Resistor_SMD:R_0805_2012Metric_Pad1.20x1.40mm_HandSolder, B.Cu at (208.8, 162.7)
- added R_5: R, Resistor_SMD:R_0805_2012Metric_Pad1.20x1.40mm_HandSolder, B.Cu at (227.8, 162.7)
- added R_6: R, Resistor_SMD:R_0805_2012Metric_Pad1.20x1.40mm_HandSolder, B.Cu at (246.9, 162.7)
- added R_7: R, Resistor_SMD:R_0805_2012Metric_Pad1.20x1.40mm_HandSolder, B.Cu at (265.9, 162.7)
- added R_8: R, Resistor_SMD:R_0805_2012Metric_Pad1.20x1.40mm_HandSolder, B.Cu at (285.0, 162.7)
- added R_9: R, Resistor_SMD:R_0805_2012Metric_Pad1.20x1.40mm_HandSolder, B.Cu at (304.0, 162.7)
- added R_Macro1: R, Resistor_SMD:R_0805_2012Metric_Pad1.20x1.40mm_HandSolder, B.Cu at (84.9, 162.7)
- added R_Macro10: R, Resistor_SMD:R_0805_2012Metric_Pad1.20x1.40mm_HandSolder, B.Cu at (104.0, 238.9)
- added R_Macro2: R, Resistor_SMD:R_0805_2012Metric_Pad1.20x1.40mm_HandSolder, B.Cu at (104.0, 162.7)
- added R_Macro3: R, Resistor_SMD:R_0805_2012Metric_Pad1.20x1.40mm_HandSolder, B.Cu at (84.9, 181.8)
- added R_Macro4: R, Resistor_SMD:R_0805_2012Metric_Pad1.20x1.40mm_HandSolder, B.Cu at (104.0, 181.8)
- added R_Macro5: R, Resistor_SMD:R_0805_2012Metric_Pad1.20x1.40mm_HandSolder, B.Cu at (84.9, 200.8)
- added R_Macro6: R, Resistor_SMD:R_0805_2012Metric_Pad1.20x1.40mm_HandSolder, B.Cu at (104.0, 200.8)
- added R_Macro7: R, Resistor_SMD:R_0805_2012Metric_Pad1.20x1.40mm_HandSolder, B.Cu at (84.9, 219.9)
- added R_Macro8: R, Resistor_SMD:R_0805_2012Metric_Pad1.20x1.40mm_HandSolder, B.Cu at (104.0, 219.9)
- added R_Macro9: R, Resistor_SMD:R_0805_2012Metric_Pad1.20x1.40mm_HandSolder, B.Cu at (84.9, 238.9)
- added R_a1: R, Resistor_SMD:R_0805_2012Metric_Pad1.20x1.40mm_HandSolder, B.Cu at (165.9, 200.8)
- added R_app1: R, Resistor_SMD:R_0805_2012Metric_Pad1.20x1.40mm_HandSolder, B.Cu at (373.1, 238.9)
- added R_b1: R, Resistor_SMD:R_0805_2012Metric_Pad1.20x1.40mm_HandSolder, B.Cu at (251.6, 219.9)
- added R_bsls1: R, Resistor_SMD:R_0805_2012Metric_Pad1.20x1.40mm_HandSolder, B.Cu at (395.3, 181.8)
- added R_bspc1: R, Resistor_SMD:R_0805_2012Metric_Pad1.20x1.40mm_HandSolder, B.Cu at (389.7, 162.7)
- added R_c1: R, Resistor_SMD:R_0805_2012Metric_Pad1.20x1.40mm_HandSolder, B.Cu at (213.5, 219.9)
- added R_caps1: R, Resistor_SMD:R_0805_2012Metric_Pad1.20x1.40mm_HandSolder, B.Cu at (139.7, 200.8)
- added R_comm1: R, Resistor_SMD:R_0805_2012Metric_Pad1.20x1.40mm_HandSolder, B.Cu at (308.8, 219.9)
- added R_d1: R, Resistor_SMD:R_0805_2012Metric_Pad1.20x1.40mm_HandSolder, B.Cu at (204.0, 200.8)
- added R_del1: R, Resistor_SMD:R_0805_2012Metric_Pad1.20x1.40mm_HandSolder, B.Cu at (427.8, 181.8)
- added R_dot1: R, Resistor_SMD:R_0805_2012Metric_Pad1.20x1.40mm_HandSolder, B.Cu at (327.8, 219.9)
- added R_down1: R, Resistor_SMD:R_0805_2012Metric_Pad1.20x1.40mm_HandSolder, B.Cu at (446.9, 238.9)
- added R_e1: R, Resistor_SMD:R_0805_2012Metric_Pad1.20x1.40mm_HandSolder, B.Cu at (199.2, 181.8)
- added R_end1: R, Resistor_SMD:R_0805_2012Metric_Pad1.20x1.40mm_HandSolder, B.Cu at (446.9, 181.8)
- added R_ent1: R, Resistor_SMD:R_0805_2012Metric_Pad1.20x1.40mm_HandSolder, B.Cu at (387.4, 200.8)
- added R_eql1: R, Resistor_SMD:R_0805_2012Metric_Pad1.20x1.40mm_HandSolder, B.Cu at (361.2, 162.7)
- added R_esc1: R, Resistor_SMD:R_0805_2012Metric_Pad1.20x1.40mm_HandSolder, B.Cu at (132.6, 134.1)
- added R_f1: R, Resistor_SMD:R_0805_2012Metric_Pad1.20x1.40mm_HandSolder, B.Cu at (170.7, 134.1)
- added R_f10: R, Resistor_SMD:R_0805_2012Metric_Pad1.20x1.40mm_HandSolder, B.Cu at (361.2, 134.1)
- added R_f11: R, Resistor_SMD:R_0805_2012Metric_Pad1.20x1.40mm_HandSolder, B.Cu at (380.2, 134.1)
- added R_f12: R, Resistor_SMD:R_0805_2012Metric_Pad1.20x1.40mm_HandSolder, B.Cu at (399.3, 134.1)
- added R_f13: R, Resistor_SMD:R_0805_2012Metric_Pad1.20x1.40mm_HandSolder, B.Cu at (223.0, 200.8)
- added R_f2: R, Resistor_SMD:R_0805_2012Metric_Pad1.20x1.40mm_HandSolder, B.Cu at (189.7, 134.1)
- added R_f3: R, Resistor_SMD:R_0805_2012Metric_Pad1.20x1.40mm_HandSolder, B.Cu at (208.8, 134.1)
- added R_f4: R, Resistor_SMD:R_0805_2012Metric_Pad1.20x1.40mm_HandSolder, B.Cu at (227.8, 134.1)
- added R_f5: R, Resistor_SMD:R_0805_2012Metric_Pad1.20x1.40mm_HandSolder, B.Cu at (256.4, 134.1)
- added R_f6: R, Resistor_SMD:R_0805_2012Metric_Pad1.20x1.40mm_HandSolder, B.Cu at (275.4, 134.1)
- added R_f7: R, Resistor_SMD:R_0805_2012Metric_Pad1.20x1.40mm_HandSolder, B.Cu at (295.3, 134.1)
- added R_f8: R, Resistor_SMD:R_0805_2012Metric_Pad1.20x1.40mm_HandSolder, B.Cu at (313.5, 134.1)
- added R_f9: R, Resistor_SMD:R_0805_2012Metric_Pad1.20x1.40mm_HandSolder, B.Cu at (342.1, 134.1)
- added R_g1: R, Resistor_SMD:R_0805_2012Metric_Pad1.20x1.40mm_HandSolder, B.Cu at (242.1, 200.8)
- added R_grv1: R, Resistor_SMD:R_0805_2012Metric_Pad1.20x1.40mm_HandSolder, B.Cu at (132.6, 162.7)
- added R_h1: R, Resistor_SMD:R_0805_2012Metric_Pad1.20x1.40mm_HandSolder, B.Cu at (261.1, 200.8)
- added R_home1: R, Resistor_SMD:R_0805_2012Metric_Pad1.20x1.40mm_HandSolder, B.Cu at (446.9, 162.7)
- added R_i1: R, Resistor_SMD:R_0805_2012Metric_Pad1.20x1.40mm_HandSolder, B.Cu at (294.5, 181.8)
- added R_ins1: R, Resistor_SMD:R_0805_2012Metric_Pad1.20x1.40mm_HandSolder, B.Cu at (427.8, 162.7)
- added R_j1: R, Resistor_SMD:R_0805_2012Metric_Pad1.20x1.40mm_HandSolder, B.Cu at (280.2, 200.8)
- added R_k1: R, Resistor_SMD:R_0805_2012Metric_Pad1.20x1.40mm_HandSolder, B.Cu at (299.2, 200.8)
- added R_l1: R, Resistor_SMD:R_0805_2012Metric_Pad1.20x1.40mm_HandSolder, B.Cu at (318.3, 200.8)
- added R_lalt1: R, Resistor_SMD:R_0805_2012Metric_Pad1.20x1.40mm_HandSolder, B.Cu at (182.6, 238.9)
- added R_lbrc1: R, Resistor_SMD:R_0805_2012Metric_Pad1.20x1.40mm_HandSolder, B.Cu at (351.6, 181.8)
- added R_lctl1: R, Resistor_SMD:R_0805_2012Metric_Pad1.20x1.40mm_HandSolder, B.Cu at (134.9, 238.9)
- added R_left1: R, Resistor_SMD:R_0805_2012Metric_Pad1.20x1.40mm_HandSolder, B.Cu at (427.8, 238.9)
- added R_lgui1: R, Resistor_SMD:R_0805_2012Metric_Pad1.20x1.40mm_HandSolder, B.Cu at (158.8, 238.9)
- added R_lsft1: R, Resistor_SMD:R_0805_2012Metric_Pad1.20x1.40mm_HandSolder, B.Cu at (144.5, 219.9)
- added R_m1: R, Resistor_SMD:R_0805_2012Metric_Pad1.20x1.40mm_HandSolder, B.Cu at (289.7, 219.9)
- added R_mins1: R, Resistor_SMD:R_0805_2012Metric_Pad1.20x1.40mm_HandSolder, B.Cu at (342.1, 162.7)
- added R_n1: R, Resistor_SMD:R_0805_2012Metric_Pad1.20x1.40mm_HandSolder, B.Cu at (270.7, 219.9)
- added R_o1: R, Resistor_SMD:R_0805_2012Metric_Pad1.20x1.40mm_HandSolder, B.Cu at (313.5, 181.8)
- added R_p1: R, Resistor_SMD:R_0805_2012Metric_Pad1.20x1.40mm_HandSolder, B.Cu at (332.6, 181.8)
- added R_paus1: R, Resistor_SMD:R_0805_2012Metric_Pad1.20x1.40mm_HandSolder, B.Cu at (465.9, 134.1)
- added R_pgdn1: R, Resistor_SMD:R_0805_2012Metric_Pad1.20x1.40mm_HandSolder, B.Cu at (465.9, 181.8)
- added R_pgup1: R, Resistor_SMD:R_0805_2012Metric_Pad1.20x1.40mm_HandSolder, B.Cu at (465.9, 162.7)
- added R_pscr1: R, Resistor_SMD:R_0805_2012Metric_Pad1.20x1.40mm_HandSolder, B.Cu at (427.8, 134.1)
- added R_q1: R, Resistor_SMD:R_0805_2012Metric_Pad1.20x1.40mm_HandSolder, B.Cu at (161.1, 181.8)
- added R_quot1: R, Resistor_SMD:R_0805_2012Metric_Pad1.20x1.40mm_HandSolder, B.Cu at (356.4, 200.8)
- added R_r1: R, Resistor_SMD:R_0805_2012Metric_Pad1.20x1.40mm_HandSolder, B.Cu at (218.3, 181.8)
- added R_ralt1: R, Resistor_SMD:R_0805_2012Metric_Pad1.20x1.40mm_HandSolder, B.Cu at (325.4, 238.9)
- added R_rbrc1: R, Resistor_SMD:R_0805_2012Metric_Pad1.20x1.40mm_HandSolder, B.Cu at (370.7, 181.8)
- added R_rctl1: R, Resistor_SMD:R_0805_2012Metric_Pad1.20x1.40mm_HandSolder, B.Cu at (396.9, 238.9)
- added R_rght1: R, Resistor_SMD:R_0805_2012Metric_Pad1.20x1.40mm_HandSolder, B.Cu at (465.9, 238.9)
- added R_rgui1: R, Resistor_SMD:R_0805_2012Metric_Pad1.20x1.40mm_HandSolder, B.Cu at (349.2, 238.9)
- added R_rsft1: R, Resistor_SMD:R_0805_2012Metric_Pad1.20x1.40mm_HandSolder, B.Cu at (382.6, 219.9)
- added R_s1: R, Resistor_SMD:R_0805_2012Metric_Pad1.20x1.40mm_HandSolder, B.Cu at (184.9, 200.8)
- added R_sclk1: R, Resistor_SMD:R_0805_2012Metric_Pad1.20x1.40mm_HandSolder, B.Cu at (446.9, 134.1)
- added R_scln1: R, Resistor_SMD:R_0805_2012Metric_Pad1.20x1.40mm_HandSolder, B.Cu at (337.3, 200.8)
- added R_slsh1: R, Resistor_SMD:R_0805_2012Metric_Pad1.20x1.40mm_HandSolder, B.Cu at (346.9, 219.9)
- added R_spc1: R, Resistor_SMD:R_0805_2012Metric_Pad1.20x1.40mm_HandSolder, B.Cu at (254.0, 238.9)
- added R_t1: R, Resistor_SMD:R_0805_2012Metric_Pad1.20x1.40mm_HandSolder, B.Cu at (237.3, 181.8)
- added R_tab1: R, Resistor_SMD:R_0805_2012Metric_Pad1.20x1.40mm_HandSolder, B.Cu at (137.3, 181.8)
- added R_u1: R, Resistor_SMD:R_0805_2012Metric_Pad1.20x1.40mm_HandSolder, B.Cu at (275.4, 181.8)
- added R_up1: R, Resistor_SMD:R_0805_2012Metric_Pad1.20x1.40mm_HandSolder, B.Cu at (446.9, 219.9)
- added R_usb1: R, Resistor_SMD:R_0805_2012Metric_Pad1.20x1.40mm_HandSolder, F.Cu at (59.5, 119.1)
- added R_usb2: 1, Resistor_SMD:R_0805_2012Metric_Pad1.20x1.40mm_HandSolder, F.Cu at (59.5, 121.4)
- added R_v2: R, Resistor_SMD:R_0805_2012Metric_Pad1.20x1.40mm_HandSolder, B.Cu at (232.6, 219.9)
- added R_w1: R, Resistor_SMD:R_0805_2012Metric_Pad1.20x1.40mm_HandSolder, B.Cu at (180.2, 181.8)
- added R_x1: R, Resistor_SMD:R_0805_2012Metric_Pad1.20x1.40mm_HandSolder, B.Cu at (194.5, 217.5)
- added R_y1: R, Resistor_SMD:R_0805_2012Metric_Pad1.20x1.40mm_HandSolder, B.Cu at (256.4, 181.8)
- added R_z1: R, Resistor_SMD:R_0805_2012Metric_Pad1.20x1.40mm_HandSolder, B.Cu at (175.4, 219.9)
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Connections:
- MX_0 pad 1: unconnected-(MX_0-Pad1) -> Col_0
- MX_1 pad 1: unconnected-(MX_1-Pad1) -> Col_1
- MX_2 pad 1: unconnected-(MX_2-Pad1) -> Col_2
- MX_3 pad 1: unconnected-(MX_3-Pad1) -> Col_3
- MX_4 pad 1: unconnected-(MX_4-Pad1) -> Col_4
- MX_5 pad 1: unconnected-(MX_5-Pad1) -> Col_5
- MX_6 pad 1: unconnected-(MX_6-Pad1) -> Col_6
- MX_7 pad 1: unconnected-(MX_7-Pad1) -> Col_7
- MX_8 pad 1: unconnected-(MX_8-Pad1) -> Col_8
- MX_9 pad 1: unconnected-(MX_9-Pad1) -> Col_9
- MX_Macro1 pad 1: unconnected-(MX_Macro1-Pad1) -> Col_8
- MX_Macro10 pad 1: unconnected-(MX_Macro10-Pad1) -> Col_7
- MX_Macro2 pad 1: unconnected-(MX_Macro2-Pad1) -> Col_9
- MX_Macro3 pad 1: unconnected-(MX_Macro3-Pad1) -> Col_7
- MX_Macro4 pad 1: unconnected-(MX_Macro4-Pad1) -> Col_8
- MX_Macro5 pad 1: unconnected-(MX_Macro5-Pad1) -> Col_6
- MX_Macro6 pad 1: unconnected-(MX_Macro6-Pad1) -> Col_7
- MX_Macro7 pad 1: unconnected-(MX_Macro7-Pad1) -> Col_1
- MX_Macro8 pad 1: unconnected-(MX_Macro8-Pad1) -> Col_2
- MX_Macro9 pad 1: unconnected-(MX_Macro9-Pad1) -> Col_6
- MX_a1 pad 1: unconnected-(MX_a1-Pad1) -> Col_9
- MX_app1 pad 1: unconnected-(MX_app1-Pad1) -> Col_4
- MX_b1 pad 1: unconnected-(MX_b1-Pad1) -> Col_8
- MX_bsls1 pad 1: unconnected-(MX_bsls1-Pad1) -> Col_2
- MX_bspc1 pad 1: unconnected-(MX_bspc1-Pad1) -> Col_3
- MX_c1 pad 1: unconnected-(MX_c1-Pad1) -> Col_6
- MX_caps1 pad 1: unconnected-(MX_caps1-Pad1) -> Col_8
- MX_comm1 pad 1: unconnected-(MX_comm1-Pad1) -> Col_1
- MX_d1 pad 1: unconnected-(MX_d1-Pad1) -> Col_1
- MX_del1 pad 1: unconnected-(MX_del1-Pad1) -> Col_3
- MX_dot1 pad 1: unconnected-(MX_dot1-Pad1) -> Col_2
- MX_down1 pad 1: unconnected-(MX_down1-Pad1) -> Col_7
- MX_e1 pad 1: unconnected-(MX_e1-Pad1) -> Col_2
- MX_end1 pad 1: unconnected-(MX_end1-Pad1) -> Col_4
- MX_ent1 pad 1: unconnected-(MX_ent1-Pad1) -> Col_0
- MX_eql1 pad 1: unconnected-(MX_eql1-Pad1) -> Col_2
- MX_esc1 pad 1: unconnected-(MX_esc1-Pad1) -> Col_2
- MX_f1 pad 1: unconnected-(MX_f1-Pad1) -> Col_3
- MX_f10 pad 1: unconnected-(MX_f10-Pad1) -> Col_2
- MX_f11 pad 1: unconnected-(MX_f11-Pad1) -> Col_3
- MX_f12 pad 1: unconnected-(MX_f12-Pad1) -> Col_4
- MX_f13 pad 1: unconnected-(MX_f13-Pad1) -> Col_2
- MX_f2 pad 1: unconnected-(MX_f2-Pad1) -> Col_4
- MX_f3 pad 1: unconnected-(MX_f3-Pad1) -> Col_5
- MX_f4 pad 1: unconnected-(MX_f4-Pad1) -> Col_6
- MX_f5 pad 1: unconnected-(MX_f5-Pad1) -> Col_7
- MX_f6 pad 1: unconnected-(MX_f6-Pad1) -> Col_8
- MX_f7 pad 1: unconnected-(MX_f7-Pad1) -> Col_9
- MX_f8 pad 1: unconnected-(MX_f8-Pad1) -> Col_0
- MX_f9 pad 1: unconnected-(MX_f9-Pad1) -> Col_1
- MX_g1 pad 1: unconnected-(MX_g1-Pad1) -> Col_3
- MX_grv1 pad 1: unconnected-(MX_grv1-Pad1) -> Col_0
- MX_h1 pad 1: unconnected-(MX_h1-Pad1) -> Col_4
- MX_home1 pad 1: unconnected-(MX_home1-Pad1) -> Col_5
- MX_i1 pad 1: unconnected-(MX_i1-Pad1) -> Col_7
- MX_ins1 pad 1: unconnected-(MX_ins1-Pad1) -> Col_4
- MX_j1 pad 1: unconnected-(MX_j1-Pad1) -> Col_5
- MX_k1 pad 1: unconnected-(MX_k1-Pad1) -> Col_6
- MX_l1 pad 1: unconnected-(MX_l1-Pad1) -> Col_7
- MX_lalt1 pad 1: unconnected-(MX_lalt1-Pad1) -> Col_0
- MX_lbrc1 pad 1: unconnected-(MX_lbrc1-Pad1) -> Col_0
- MX_lctl1 pad 1: unconnected-(MX_lctl1-Pad1) -> Col_8
- MX_left1 pad 1: unconnected-(MX_left1-Pad1) -> Col_6
- MX_lgui1 pad 1: unconnected-(MX_lgui1-Pad1) -> Col_9
- MX_lsft1 pad 1: unconnected-(MX_lsft1-Pad1) -> Col_3
- MX_m1 pad 1: unconnected-(MX_m1-Pad1) -> Col_0
- MX_mins1 pad 1: unconnected-(MX_mins1-Pad1) -> Col_1
- MX_n1 pad 1: unconnected-(MX_n1-Pad1) -> Col_9
- MX_o1 pad 1: unconnected-(MX_o1-Pad1) -> Col_8
- MX_p1 pad 1: unconnected-(MX_p1-Pad1) -> Col_9
- MX_paus1 pad 1: unconnected-(MX_paus1-Pad1) -> Col_7
- MX_pgdn1 pad 1: unconnected-(MX_pgdn1-Pad1) -> Col_5
- MX_pgup1 pad 1: unconnected-(MX_pgup1-Pad1) -> Col_6
- MX_pscr1 pad 1: unconnected-(MX_pscr1-Pad1) -> Col_5
- MX_q1 pad 1: unconnected-(MX_q1-Pad1) -> Col_0
- MX_quot1 pad 1: unconnected-(MX_quot1-Pad1) -> Col_9
- MX_r1 pad 1: unconnected-(MX_r1-Pad1) -> Col_3
- MX_ralt1 pad 1: unconnected-(MX_ralt1-Pad1) -> Col_2
- MX_rbrc1 pad 1: unconnected-(MX_rbrc1-Pad1) -> Col_1
- MX_rctl1 pad 1: unconnected-(MX_rctl1-Pad1) -> Col_5
- MX_rght1 pad 1: unconnected-(MX_rght1-Pad1) -> Col_8
- MX_rgui1 pad 1: unconnected-(MX_rgui1-Pad1) -> Col_3
- MX_rsft1 pad 1: unconnected-(MX_rsft1-Pad1) -> Col_4
- MX_s1 pad 1: unconnected-(MX_s1-Pad1) -> Col_0
- MX_sclk1 pad 1: unconnected-(MX_sclk1-Pad1) -> Col_6
- MX_scln1 pad 1: unconnected-(MX_scln1-Pad1) -> Col_8
- MX_slsh1 pad 1: unconnected-(MX_slsh1-Pad1) -> Col_3
- MX_spc1 pad 1: unconnected-(MX_spc1-Pad1) -> Col_1
- MX_t1 pad 1: unconnected-(MX_t1-Pad1) -> Col_4
- MX_tab1 pad 1: unconnected-(MX_tab1-Pad1) -> Col_9
- MX_u1 pad 1: unconnected-(MX_u1-Pad1) -> Col_6
- MX_up1 pad 1: unconnected-(MX_up1-Pad1) -> Col_5
- MX_v1 pad 1: unconnected-(MX_v1-Pad1) -> Col_7
- MX_w1 pad 1: unconnected-(MX_w1-Pad1) -> Col_1
- MX_x1 pad 1: unconnected-(MX_x1-Pad1) -> Col_5
- MX_y1 pad 1: unconnected-(MX_y1-Pad1) -> Col_5
- MX_z1 pad 1: unconnected-(MX_z1-Pad1) -> Col_4
- SW_re1 pad S2: Row_0 -> Net-(D_re1-Pad2)
- SW_re2 pad S2: Row_0 -> Net-(D_re2-Pad2)
- U1 pad 2: unconnected-(U1-Pad2) -> RO_1_DN
- USB1 pad 11: V_USB_IN -> LED_VIN
- USB1 pad 2: V_USB_IN -> LED_VIN
Routing:
- net LED_VIN: track 0.00 -> 2510.7 mm, vias 0 -> 6
- net Col_0: track 0.00 -> 1019.3 mm, vias 0 -> 4
- net Col_3: track 0.00 -> 959.2 mm, vias 0 -> 4
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Other:
- board outline added: 432.6 x 128.6 mm
